Commit message: Changes to be committed: 	modified:   turtlebot3_description/urdf/turtlebot3_burger.gazebo.xacro 	modified:   turtlebot3_description/urdf/turtlebot3_burger.urdf.xacro 	modified:   turtlebot3_teleop/launch/turtlebot3_teleop_key.launch

File: turtlebot3_description/urdf/turtlebot3_burger.gazebo.xacro (robot description, xacro)
@@ -3,8 +3,18 @@
   <xacro:arg name="laser_visual" default="false"/>
   <xacro:arg name="imu_visual"   default="false"/>
-  <gazebo reference="base_link">
-    <material>Gazebo/DarkGrey</material>
-  </gazebo>
-  <gazebo reference="wheel_left_link">
+ <gazebo reference="base_link_$(arg number)">
+      <material>Gazebo/DarkGrey</material>
+    <sensor type="contact" name="collision_base_$(arg number)">
+       <plugin name="collision_plugin" filename="libgazebo_ros_bumper2.so">
+       <bumperTopicName>bump</bumperTopicName>
+          <frameName>base_link_$(arg number)</frameName>
+        </plugin>
+         <contact>
+          <collision>base_footprint_$(arg number)_fixed_joint_lump__base_col_collision</collision>
+      </contact>
+              <update_rate> 100 </update_rate>
+  </sensor>
+</gazebo>
+  <gazebo reference="wheel_left_link_$(arg number)">
     <mu1>0.1</mu1>
     <mu2>0.1</mu2>
@@ -15,6 +25,16 @@
     <fdir1>1 0 0</fdir1>
     <material>Gazebo/FlatBlack</material>
+     <sensor type="contact" name="collision_lw_$(arg number)">
+       <plugin name="collision_plugin" filename="libgazebo_ros_bumper2.so">
+       <bumperTopicName>bump</bumperTopicName>
+          <frameName>base_link_$(arg number)</frameName>
+        </plugin>
+         <contact>
+          <collision>wheel_left_link_$(arg number)_collision</collision>
+      </contact>
+              <update_rate> 100 </update_rate>
+  </sensor>
   </gazebo>
-  <gazebo reference="wheel_right_link">
+  <gazebo reference="wheel_right_link_$(arg number)">
     <mu1>0.1</mu1>
     <mu2>0.1</mu2>
@@ -25,6 +45,16 @@
     <fdir1>1 0 0</fdir1>
     <material>Gazebo/FlatBlack</material>
+     <sensor type="contact" name="collision_rw_$(arg number)">
+       <plugin name="collision_plugin" filename="libgazebo_ros_bumper2.so">
+       <bumperTopicName>bump</bumperTopicName>
+          <frameName>base_link_$(arg number)</frameName>
+        </plugin>
+         <contact>
+          <collision>wheel_right_link_$(arg number)_collision</collision>
+      </contact>
+              <update_rate> 100 </update_rate>
+  </sensor>
   </gazebo>
-  <gazebo reference="caster_back_link">
+  <gazebo reference="caster_back_link_$(arg number)">
     <mu1>0.1</mu1>
     <mu2>0.1</mu2>
@@ -35,6 +65,6 @@
     <material>Gazebo/FlatBlack</material>
   </gazebo>
-  <gazebo reference="imu_link">
-    <sensor type="imu" name="imu">
+  <gazebo reference="imu_link_$(arg number)">
+    <sensor type="imu" name="imu_$(arg number)">
       <always_on>true</always_on>
       <visualize>$(arg imu_visual)</visualize>
@@ -43,5 +73,5 @@
   </gazebo>
   <gazebo>
-    <plugin name="turtlebot3_burger_controller" filename="libgazebo_ros_diff_drive.so">
+    <plugin name="turtlebot3_burger_controller_$(arg number)" filename="libgazebo_ros_diff_drive.so">
       <commandTopic>cmd_vel</commandTopic>
       <odometryTopic>odom</odometryTopic>
@@ -49,5 +79,5 @@
       <odometrySource>world</odometrySource>
       <publishOdomTF>true</publishOdomTF>
-      <robotBaseFrame>base_footprint</robotBaseFrame>
+      <robotBaseFrame>base_footprint_$(arg number)</robotBaseFrame>
       <publishWheelTF>false</publishWheelTF>
       <publishTf>true</publishTf>
@@ -55,6 +85,6 @@
       <legacyMode>false</legacyMode>
       <updateRate>30</updateRate>
-      <leftJoint>wheel_left_joint</leftJoint>
-      <rightJoint>wheel_right_joint</rightJoint>
+      <leftJoint>wheel_left_joint_$(arg number)</leftJoint>
+      <rightJoint>wheel_right_joint_$(arg number)</rightJoint>
       <wheelSeparation>0.160</wheelSeparation>
       <wheelDiameter>0.066</wheelDiameter>
@@ -64,13 +94,14 @@
     </plugin>
   </gazebo>
+<!--
   <gazebo>
-    <plugin name="imu_plugin" filename="libgazebo_ros_imu.so">
+    <plugin name="imu_plugin_$(arg number)" filename="libgazebo_ros_imu.so">
       <alwaysOn>true</alwaysOn>
-      <bodyName>imu_link</bodyName>
-      <frameName>imu_link</frameName>
+      <bodyName>imu_link_$(arg number)</bodyName>
+      <frameName>imu_link_$(arg number)</frameName>
       <topicName>imu</topicName>
       <serviceName>imu_service</serviceName>
-      <gaussianNoise>0.0</gaussianNoise>
-      <updateRate>0</updateRate>
+      <gaussianNoise>0.001</gaussianNoise>
+      <updateRate>100</updateRate>
       <imu>
         <noise>
@@ -92,7 +123,22 @@
     </plugin>
   </gazebo>
-  <gazebo reference="base_scan">
+-->
+  <gazebo>
+    <plugin name="imu_controller" filename="libhector_gazebo_ros_imu.so">
+      <robotNamespace>burger_$(arg number)</robotNamespace>
+      <updateRate>50.0</updateRate>
+      <bodyName>imu_link_$(arg number)</bodyName>
+      <topicName>imu</topicName>
+      <accelDrift>0.005 0.005 0.005</accelDrift>
+      <accelGaussianNoise>0.01 0.01 0.01</accelGaussianNoise>
+      <rateDrift>0.005 0.005 0.005 </rateDrift>
+      <rateGaussianNoise>0.005 0.005 0.005 </rateGaussianNoise>
+      <headingDrift>0.005</headingDrift>
+      <headingGaussianNoise>0.005</headingGaussianNoise>
+    </plugin>
+  </gazebo>
+  <gazebo reference="base_scan_$(arg number)">
     <material>Gazebo/FlatBlack</material>
-    <sensor type="ray" name="lds_lfcd_sensor">
+    <sensor type="ray" name="lds_lfcd_sensor_$(arg number)">
       <pose>0 0 0 0 0 0</pose>
       <visualize>$(arg laser_visual)</visualize>
@@ -118,9 +164,25 @@
         </noise>
       </ray>
-      <plugin name="gazebo_ros_lds_lfcd_controller" filename="libgazebo_ros_laser.so">
+      <plugin name="gazebo_ros_lds_lfcd_controller_$(arg number)" filename="libgazebo_ros_laser.so">
         <topicName>scan</topicName>
-        <frameName>base_scan</frameName>
+        <frameName>base_scan_$(arg number)</frameName>
       </plugin>
     </sensor>
   </gazebo>
+   <gazebo>
+    <plugin name="magnetic_controller" filename="libhector_gazebo_ros_magnetic.so">
+      <robotNamespace>burger_$(arg number)</robotNamespace>
+      <updateRate>50.0</updateRate>
+      <bodyName>imu_link_$(arg number)</bodyName>
+      <topicName>magnetic</topicName>
+      <referenceHeading>0.0</referenceHeading>
+      <declination>0.0</declination>
+      <inclination>60.0</inclination>
+      <magnitude> 1.2 </magnitude>
+      <offset>0 0 0</offset>
+       <driftFrequency>0.005 0.005 0.005</driftFrequency>
+      <gaussianNoise>0.01 0.01 0.01</gaussianNoise>
+      <useMagneticFieldMsgs>false</useMagneticFieldMsgs>
+    </plugin>
+  </gazebo>
 </robot>

File: turtlebot3_description/urdf/turtlebot3_burger.urdf.xacro (robot description, xacro)
@@ -1,13 +1,15 @@
 <?xml version="1.0" ?>
-<robot name="turtlebot3_burger" xmlns:xacro="http://ros.org/wiki/xacro">
-  <xacro:include filename="$(find turtlebot3_description)/urdf/common_properties.xacro"/>
+<robot name="turtlebot3_burger"
+  xmlns:xacro="http://ros.org/wiki/xacro" >
+ <xacro:arg name="number" default=""/>
+ <xacro:include filename="$(find turtlebot3_description)/urdf/common_properties.xacro"/>
   <xacro:include filename="$(find turtlebot3_description)/urdf/turtlebot3_burger.gazebo.xacro"/>
-  <link name="base_footprint"/>
-  <joint name="base_joint" type="fixed">
-    <parent link="base_footprint"/>
-    <child link="base_link"/>
+  <link name="base_footprint_$(arg number)"/>
+  <joint name="base_joint_$(arg number)" type="fixed">
+    <parent link="base_footprint_$(arg number)"/>
+    <child link="base_link_$(arg number)"/>
     <origin xyz="0.0 0.0 0.010" rpy="0 0 0"/>
   </joint>
-  <link name="base_link">
+  <link name="base_link_$(arg number)">
     <visual>
       <origin xyz="-0.032 0 0.0" rpy="0 0 0"/>
@@ -17,5 +19,5 @@
       <material name="light_black"/>
     </visual>
-    <collision>
+    <collision name="base_col">
       <origin xyz="-0.032 0 0.070" rpy="0 0 0"/>
       <geometry>
@@ -31,11 +33,11 @@
     </inertial>
   </link>
-  <joint name="wheel_left_joint" type="continuous">
-    <parent link="base_link"/>
-    <child link="wheel_left_link"/>
+  <joint name="wheel_left_joint_$(arg number)" type="continuous">
+    <parent link="base_link_$(arg number)"/>
+    <child link="wheel_left_link_$(arg number)"/>
     <origin xyz="0.0 0.08 0.023" rpy="-1.57 0 0"/>
     <axis xyz="0 0 1"/>
   </joint>
-  <link name="wheel_left_link">
+  <link name="wheel_left_link_$(arg number)">
     <visual>
       <origin xyz="0 0 0" rpy="1.57 0 0"/>
@@ -59,11 +61,11 @@
       </inertial>
   </link>
-  <joint name="wheel_right_joint" type="continuous">
-    <parent link="base_link"/>
-    <child link="wheel_right_link"/>
+  <joint name="wheel_right_joint_$(arg number)" type="continuous">
+    <parent link="base_link_$(arg number)"/>
+    <child link="wheel_right_link_$(arg number)"/>
     <origin xyz="0.0 -0.080 0.023" rpy="-1.57 0 0"/>
     <axis xyz="0 0 1"/>
   </joint>
-  <link name="wheel_right_link">
+  <link name="wheel_right_link_$(arg number)">
     <visual>
       <origin xyz="0 0 0" rpy="1.57 0 0"/>
@@ -87,10 +89,10 @@
       </inertial>
   </link>
-  <joint name="caster_back_joint" type="fixed">
-    <parent link="base_link"/>
-    <child link="caster_back_link"/>
+  <joint name="caster_back_joint_$(arg number)" type="fixed">
+    <parent link="base_link_$(arg number)"/>
+    <child link="caster_back_link_$(arg number)"/>
     <origin xyz="-0.081 0 -0.004" rpy="-1.57 0 0"/>
   </joint>
-  <link name="caster_back_link">
+  <link name="caster_back_link_$(arg number)">
     <collision>
       <origin xyz="0 0.001 0" rpy="0 0 0"/>
@@ -107,16 +109,16 @@
     </inertial>
   </link>
-  <joint name="imu_joint" type="fixed">
-    <parent link="base_link"/>
-    <child link="imu_link"/>
+  <joint name="imu_joint_$(arg number)" type="fixed">
+    <parent link="base_link_$(arg number)"/>
+    <child link="imu_link_$(arg number)"/>
     <origin xyz="-0.032 0 0.068" rpy="0 0 0"/>
   </joint>
-  <link name="imu_link"/>
-  <joint name="scan_joint" type="fixed">
-    <parent link="base_link"/>
-    <child link="base_scan"/>
+  <link name="imu_link_$(arg number)"/>
+  <joint name="scan_joint_$(arg number)" type="fixed">
+    <parent link="base_link_$(arg number)"/>
+    <child link="base_scan_$(arg number)"/>
     <origin xyz="-0.032 0 0.172" rpy="0 0 0"/>
   </joint>
-  <link name="base_scan">
+  <link name="base_scan_$(arg number)">
     <visual>
       <origin xyz="0 0 0.0" rpy="0 0 0"/>

Commit message: naming

File: turtlebot3_description/urdf/turtlebot3_burger.gazebo.xacro (robot description, xacro)
@@ -76,5 +76,5 @@
       <commandTopic>cmd_vel</commandTopic>
       <odometryTopic>odom</odometryTopic>
-      <odometryFrame>odom</odometryFrame>
+      <odometryFrame>odom_burger$(arg number)</odometryFrame>
       <odometrySource>world</odometrySource>
       <publishOdomTF>true</publishOdomTF>

File: turtlebot3_description/urdf/turtlebot3_burger.urdf.xacro (robot description, xacro)
@@ -6,9 +6,4 @@
   <xacro:include filename="$(find turtlebot3_description)/urdf/turtlebot3_burger.gazebo.xacro"/>
   <link name="base_footprint_$(arg number)"/>
-  <joint name="base_joint_$(arg number)" type="fixed">
-    <parent link="base_footprint_$(arg number)"/>
-    <child link="base_link_$(arg number)"/>
-    <origin xyz="0.0 0.0 0.010" rpy="0 0 0"/>
-  </joint>
   <link name="base_link_$(arg number)">
     <visual>
@@ -33,10 +28,4 @@
     </inertial>
   </link>
-  <joint name="wheel_left_joint_$(arg number)" type="continuous">
-    <parent link="base_link_$(arg number)"/>
-    <child link="wheel_left_link_$(arg number)"/>
-    <origin xyz="0.0 0.08 0.023" rpy="-1.57 0 0"/>
-    <axis xyz="0 0 1"/>
-  </joint>
   <link name="wheel_left_link_$(arg number)">
     <visual>
@@ -61,10 +50,4 @@
       </inertial>
   </link>
-  <joint name="wheel_right_joint_$(arg number)" type="continuous">
-    <parent link="base_link_$(arg number)"/>
-    <child link="wheel_right_link_$(arg number)"/>
-    <origin xyz="0.0 -0.080 0.023" rpy="-1.57 0 0"/>
-    <axis xyz="0 0 1"/>
-  </joint>
   <link name="wheel_right_link_$(arg number)">
     <visual>
@@ -89,9 +72,4 @@
       </inertial>
   </link>
-  <joint name="caster_back_joint_$(arg number)" type="fixed">
-    <parent link="base_link_$(arg number)"/>
-    <child link="caster_back_link_$(arg number)"/>
-    <origin xyz="-0.081 0 -0.004" rpy="-1.57 0 0"/>
-  </joint>
   <link name="caster_back_link_$(arg number)">
     <collision>
@@ -109,15 +87,5 @@
     </inertial>
   </link>
-  <joint name="imu_joint_$(arg number)" type="fixed">
-    <parent link="base_link_$(arg number)"/>
-    <child link="imu_link_$(arg number)"/>
-    <origin xyz="-0.032 0 0.068" rpy="0 0 0"/>
-  </joint>
   <link name="imu_link_$(arg number)"/>
-  <joint name="scan_joint_$(arg number)" type="fixed">
-    <parent link="base_link_$(arg number)"/>
-    <child link="base_scan_$(arg number)"/>
-    <origin xyz="-0.032 0 0.172" rpy="0 0 0"/>
-  </joint>
   <link name="base_scan_$(arg number)">
     <visual>
@@ -142,3 +110,35 @@
     </inertial>
   </link>
+ <joint name="base_joint_$(arg number)" type="fixed">
+    <parent link="base_footprint_$(arg number)"/>
+    <child link="base_link_$(arg number)"/>
+    <origin xyz="0.0 0.0 0.010" rpy="0 0 0"/>
+  </joint>
+  <joint name="wheel_left_joint_$(arg number)" type="continuous">
+    <parent link="base_link_$(arg number)"/>
+    <child link="wheel_left_link_$(arg number)"/>
+    <origin xyz="0.0 0.08 0.023" rpy="-1.57 0 0"/>
+    <axis xyz="0 0 1"/>
+  </joint>
+  <joint name="wheel_right_joint_$(arg number)" type="continuous">
+    <parent link="base_link_$(arg number)"/>
+    <child link="wheel_right_link_$(arg number)"/>
+    <origin xyz="0.0 -0.080 0.023" rpy="-1.57 0 0"/>
+    <axis xyz="0 0 1"/>
+  </joint>
+  <joint name="caster_back_joint_$(arg number)" type="fixed">
+    <parent link="base_link_$(arg number)"/>
+    <child link="caster_back_link_$(arg number)"/>
+    <origin xyz="-0.081 0 -0.004" rpy="-1.57 0 0"/>
+  </joint>
+  <joint name="imu_joint_$(arg number)" type="fixed">
+    <parent link="base_link_$(arg number)"/>
+    <child link="imu_link_$(arg number)"/>
+    <origin xyz="-0.032 0 0.068" rpy="0 0 0"/>
+  </joint>
+  <joint name="scan_joint_$(arg number)" type="fixed">
+    <parent link="base_link_$(arg number)"/>
+    <child link="base_scan_$(arg number)"/>
+    <origin xyz="-0.032 0 0.172" rpy="0 0 0"/>
+  </joint>
 </robot>
